Commit message: Operator<< for FT sensor, updated centauro config files

File: IXBotInterface/configs/urdf/centauro.urdf (robot description, URDF)
Before this commit: robot centauro, 17 links, 16 joints
Links:
- added link ft_foot_1, mass 0.001; visual box size=0.01 0.01 0.01
- added link ft_foot_2, mass 0.001; visual box size=0.01 0.01 0.01
- added link ft_foot_3, mass 0.001; visual box size=0.01 0.01 0.01
- added link ft_foot_4, mass 0.001; visual box size=0.01 0.01 0.01
- added link hip1_1, mass 2.0; collision box size=0.05 0.05 0.15; visual box size=0.05 0.05 0.2
- added link hip1_2, mass 2.0; collision box size=0.05 0.05 0.15; visual box size=0.05 0.05 0.2
- added link hip1_3, mass 2.0; collision box size=0.05 0.05 0.15; visual box size=0.05 0.05 0.2
- added link hip1_4, mass 2.0; collision box size=0.05 0.05 0.15; visual box size=0.05 0.05 0.2
- added link hip2_1, mass 4.5; collision box size=0.05 0.05 0.3; visual box size=0.05 0.05 0.35
- added link hip2_2, mass 4.5; collision box size=0.05 0.05 0.3; visual box size=0.05 0.05 0.35
- added link hip2_3, mass 4.5; collision box size=0.05 0.05 0.3; visual box size=0.05 0.05 0.35
- added link hip2_4, mass 4.5; collision box size=0.05 0.05 0.3; visual box size=0.05 0.05 0.35
- added link knee_1, mass 3.5; collision box size=0.05 0.05 0.2; collision sphere radius=0.05
- added link knee_2, mass 3.5; collision box size=0.05 0.05 0.2; collision sphere radius=0.05
- added link knee_3, mass 3.5; collision box size=0.05 0.05 0.2; collision sphere radius=0.05
- added link knee_4, mass 3.5; collision box size=0.05 0.05 0.2; collision sphere radius=0.05
Joints:
- added joint ft_foot_1_joint: type fixed, parent knee_1, child ft_foot_1, origin xyz=0 0 -0.3 rpy=0 0 0
- added joint ft_foot_2_joint: type fixed, parent knee_2, child ft_foot_2, origin xyz=0 0 -0.3 rpy=0 0 0
- added joint ft_foot_3_joint: type fixed, parent knee_3, child ft_foot_3, origin xyz=0 0 -0.3 rpy=0 0 0
- added joint ft_foot_4_joint: type fixed, parent knee_4, child ft_foot_4, origin xyz=0 0 -0.3 rpy=0 0 0
- added joint hip_pitch_1: type revolute, parent hip1_1, child hip2_1, origin xyz=0 0 -0.2, axis 0 -1 0, limit lower=-3.14 upper=3.14 effort=350 velocity=6.5
- added joint hip_pitch_2: type revolute, parent hip1_2, child hip2_2, origin xyz=0 0 -0.2, axis 0 1 0, limit lower=-3.14 upper=3.14 effort=350 velocity=6.5
- added joint hip_pitch_3: type revolute, parent hip1_3, child hip2_3, origin xyz=0 0 -0.2, axis 0 1 0, limit lower=-3.14 upper=3.14 effort=350 velocity=6.5
- added joint hip_pitch_4: type revolute, parent hip1_4, child hip2_4, origin xyz=0 0 -0.2, axis 0 -1 0, limit lower=-3.14 upper=3.14 effort=350 velocity=6.5
- added joint hip_yaw_1: type revolute, parent pelvis, child hip1_1, origin xyz=0.3 0.15 0 rpy=0 0 1.5707963268, axis 0 0 -1, limit lower=-2.09 upper=2.09 effort=350 velocity=6.5
- added joint hip_yaw_2: type revolute, parent pelvis, child hip1_2, origin xyz=0.3 -0.15 0 rpy=0 0 1.5707963268, axis 0 0 1, limit lower=-2.09 upper=2.09 effort=350 velocity=6.5
- added joint hip_yaw_3: type revolute, parent pelvis, child hip1_3, origin xyz=-0.3 -0.15 0 rpy=0 0 1.5707963268, axis 0 0 1, limit lower=-2.09 upper=2.09 effort=350 velocity=6.5
- added joint hip_yaw_4: type revolute, parent pelvis, child hip1_4, origin xyz=-0.3 0.15 0 rpy=0 0 1.5707963268, axis 0 0 -1, limit lower=-2.09 upper=2.09 effort=350 velocity=6.5
- added joint knee_pitch_1: type revolute, parent hip2_1, child knee_1, origin xyz=0 0 -0.35, axis 0 -1 0, limit lower=-3.14 upper=3.14 effort=35000 velocity=600.5
- added joint knee_pitch_2: type revolute, parent hip2_2, child knee_2, origin xyz=0 0 -0.35, axis 0 1 0, limit lower=-3.14 upper=3.14 effort=35000 velocity=600.5
- added joint knee_pitch_3: type revolute, parent hip2_3, child knee_3, origin xyz=0 0 -0.35, axis 0 1 0, limit lower=-3.14 upper=3.14 effort=35000 velocity=600.5
- added joint knee_pitch_4: type revolute, parent hip2_4, child knee_4, origin xyz=0 0 -0.35, axis 0 -1 0, limit lower=-3.14 upper=3.14 effort=35000 velocity=600.5
- joint j_arm1_2: origin xyz=0 0.1 0 -> xyz=-0.09115 0.06106 0.010766
- joint j_arm1_3: origin xyz=0 0 -0.2 -> xyz=0.09115 0 -0.21915
- joint j_arm1_4: origin xyz=0 0 -0.15 -> xyz=0.040 0.05615 -0.074
- joint j_arm1_5: origin xyz=0 0 -0.13 -> xyz=-0.015 -0.05615 -0.061
- joint j_arm1_6: origin xyz=0 0 -0.10 -> xyz=0 0.049 -0.180
- joint j_arm1_7: origin xyz=0 0 -0.13 -> xyz=0 -0.049 -0.169
- joint j_arm2_2: origin xyz=0 -0.1 0 -> xyz=-0.09115 -0.06106 0.010766
- joint j_arm2_3: origin xyz=0 0 -0.2 -> xyz=0.09115 0 -0.21915
- joint j_arm2_4: origin xyz=0 0 -0.15 -> xyz=0.040 -0.05615 -0.074
- joint j_arm2_5: origin xyz=0 0 -0.13 -> xyz=-0.015 0.05615 -0.061
- joint j_arm2_6: origin xyz=0 0 -0.10 -> xyz=0 -0.049 -0.180
- joint j_arm2_7: origin xyz=0 0 -0.13 -> xyz=0 0.049 -0.169
- joint reference: type fixed -> floating
