Commit message: bigman config and URDF/SRDF updated. bigman urdf added: fixed hand or not.

File: IXBotInterface/configs/srdf/bigman_config.srdf.xacro (robot description, xacro)
@@ -13,6 +13,6 @@
     <xacro:property name="BIGMAN_LEFT_ARM" value="true" />
     <xacro:property name="BIGMAN_RIGHT_ARM" value="true" />
-    <xacro:property name="BIGMAN_LEFT_HAND" value="true" />
-    <xacro:property name="BIGMAN_RIGHT_HAND" value="true" />
+    <xacro:property name="BIGMAN_LEFT_HAND" value="false" />
+    <xacro:property name="BIGMAN_RIGHT_HAND" value="false" />
     <xacro:property name="BIGMAN_TORSO" value="true" />
     <xacro:property name="BIGMAN_LEFT_LEG" value="true" />

File: IXBotInterface/configs/urdf/bigman_fixed_hands.urdf (robot description, URDF)
Before this commit: robot bigman, 73 links, 72 joints
Links:
- added link LSoftHandLink, mass 1.2; collision mesh filename=package://bigman_urdf/meshes/simple/SoftHandOpen.STL scale=0.001 -0.001 0.001; visual mesh filename=package://bigman_urdf/meshes/SoftHandOpen.STL scale=0.001 -0.001 0.001
- added link RSoftHandLink, mass 1.2; collision mesh filename=package://bigman_urdf/meshes/simple/SoftHandOpen.STL scale=0.001 0.001 0.001; visual mesh filename=package://bigman_urdf/meshes/SoftHandOpen.STL scale=0.001 0.001 0.001
- added link l_hand_lower_left_link
- added link l_hand_lower_right_link
- added link l_hand_upper_left_link
- added link l_hand_upper_right_link
- added link r_hand_lower_left_link
- added link r_hand_lower_right_link
- added link r_hand_upper_left_link
- added link r_hand_upper_right_link
- link LSoftHand: mass 1.2 -> None; geometry 
- link RSoftHand: mass 1.2 -> None; geometry 
Joints:
- added joint l_handj2: type fixed, parent LSoftHandLink, child LSoftHand, origin xyz=0 -0.0305 -0.21 rpy=0 0 0
- added joint l_handj3: type fixed, parent LSoftHand, child l_hand_upper_right_link, origin xyz=0.05 0.0 0.0 rpy=0 0 0
- added joint l_handj4: type fixed, parent LSoftHand, child l_hand_lower_right_link, origin xyz=-0.05 0.0 0.0 rpy=0 0 0
- added joint l_handj5: type fixed, parent LSoftHand, child l_hand_upper_left_link, origin xyz=0.05 0.0 0.1 rpy=0 0 0
- added joint l_handj6: type fixed, parent LSoftHand, child l_hand_lower_left_link, origin xyz=-0.05 0.0 0.1 rpy=0 0 0
- added joint r_handj2: type fixed, parent RSoftHandLink, child RSoftHand, origin xyz=0 0.0305 -0.21 rpy=0 0 0
- added joint r_handj3: type fixed, parent RSoftHand, child r_hand_upper_right_link, origin xyz=0.05 0.0 0.0 rpy=0 0 0
- added joint r_handj4: type fixed, parent RSoftHand, child r_hand_lower_right_link, origin xyz=-0.05 0.0 0.0 rpy=0 0 0
- added joint r_handj5: type fixed, parent RSoftHand, child r_hand_upper_left_link, origin xyz=0.05 0.0 0.1 rpy=0 0 0
- added joint r_handj6: type fixed, parent RSoftHand, child r_hand_lower_left_link, origin xyz=-0.05 0.0 0.1 rpy=0 0 0
- joint LAnkLat: limit lower=-0.785 upper=0.785 effort=210 velocity=6.283 -> lower=-0.785 upper=0.785 effort=120 velocity=6.283
- joint LAnkSag: limit lower=-1.39556 upper=0.697778 effort=330 velocity=6.283 -> lower=-1.39556 upper=0.697778 effort=220 velocity=6.283
- joint LElbj: limit lower=-2.96705972838 upper=0.593411945677 effort=120 velocity=6.283 -> lower=-2.96705972838 upper=0.593411945677 effort=60 velocity=6.283
- joint LHipLat: limit lower=-0.697778 upper=0.87222 effort=400 velocity=6.283 -> lower=-0.697778 upper=0.87222 effort=220 velocity=6.283
- joint LHipSag: limit lower=-2.09333 upper=1.046667 effort=400 velocity=6.283 -> lower=-2.09333 upper=1.046667 effort=220 velocity=6.283
- joint LHipYaw: limit lower=-0.872222 upper=1.57 effort=140 velocity=6.283 -> lower=-0.872222 upper=1.57 effort=120 velocity=6.283
- joint LKneeSag: limit lower=0.0 upper=2.442222 effort=400 velocity=6.283 -> lower=0.0 upper=2.442222 effort=220 velocity=6.283
- joint NeckPitchj: origin xyz=0 0 0.117 rpy=0 0 0 -> xyz=0 0 0.1155 rpy=0 0 0
- joint RAnkLat: limit lower=-0.785 upper=0.785 effort=210 velocity=6.283 -> lower=-0.785 upper=0.785 effort=120 velocity=6.283
- joint RAnkSag: limit lower=-1.39556 upper=0.697778 effort=330 velocity=6.283 -> lower=-1.39556 upper=0.697778 effort=220 velocity=6.283
- joint RElbj: limit lower=-2.96705972838 upper=0.593411945677 effort=120 velocity=6.283 -> lower=-2.96705972838 upper=0.593411945677 effort=60 velocity=6.283
- joint RHipLat: limit lower=-0.87222 upper=0.697778 effort=400 velocity=6.283 -> lower=-0.87222 upper=0.697778 effort=220 velocity=6.283
- joint RHipSag: limit lower=-2.09333 upper=1.046667 effort=400 velocity=6.283 -> lower=-2.09333 upper=1.046667 effort=220 velocity=6.283
- joint RHipYaw: limit lower=-1.57 upper=0.872222 effort=140 velocity=6.283 -> lower=-1.57 upper=0.872222 effort=120 velocity=6.283
- joint RKneeSag: limit lower=0.0 upper=2.442222 effort=400 velocity=6.283 -> lower=0.0 upper=2.442222 effort=220 velocity=6.283
- joint l_handj: axis -1 0 0 -> (none); child LSoftHand -> LSoftHandLink; limit lower=0 upper=5.0 effort=5 velocity=4.0 -> (none); origin xyz=0 0 -0.04 rpy=0 0 0 -> xyz=0 0 0 rpy=0 0 0; type revolute -> fixed
- joint r_handj: axis 1 0 0 -> (none); child RSoftHand -> RSoftHandLink; limit lower=0.0 upper=5.0 effort=5 velocity=4.0 -> (none); origin xyz=0 0 -0.04 rpy=0 0 0 -> xyz=0 0 0 rpy=0 0 0; type revolute -> fixed

Commit message: Reorganizing WALKMAN config files

File: IXBotInterface/configs/srdf/bigman_config.srdf.xacro (robot description, xacro)
@@ -16,10 +16,10 @@
     <xacro:property name="BIGMAN_RIGHT_HAND" value="false" />
     <xacro:property name="BIGMAN_TORSO" value="true" />
-    <xacro:property name="BIGMAN_LEFT_LEG" value="true" />
-    <xacro:property name="BIGMAN_RIGHT_LEG" value="true" />
+    <xacro:property name="BIGMAN_LEFT_LEG" value="false" />
+    <xacro:property name="BIGMAN_RIGHT_LEG" value="false" />
     <xacro:property name="BIGMAN_LEFT_ARM_FT" value="true" />
     <xacro:property name="BIGMAN_RIGHT_ARM_FT" value="true" />
-    <xacro:property name="BIGMAN_LEFT_LEG_FT" value="true" />
-    <xacro:property name="BIGMAN_RIGHT_LEG_FT" value="true" />
+    <xacro:property name="BIGMAN_LEFT_LEG_FT" value="false" />
+    <xacro:property name="BIGMAN_RIGHT_LEG_FT" value="false" />
     <!-- Robot kinematic chains -->
     <!-- CONSTRAINT: specify the chain inside a group: only one chain per group -->

Commit message: updated srdf_advr namespace and using proper URDF and SRDF for the WALKMAN upper body

File: IXBotInterface/configs/srdf/bigman_config.srdf.xacro (robot description, xacro)
@@ -13,6 +13,6 @@
     <xacro:property name="BIGMAN_LEFT_ARM" value="true" />
     <xacro:property name="BIGMAN_RIGHT_ARM" value="true" />
-    <xacro:property name="BIGMAN_LEFT_HAND" value="false" />
-    <xacro:property name="BIGMAN_RIGHT_HAND" value="false" />
+    <xacro:property name="BIGMAN_LEFT_HAND" value="true" />
+    <xacro:property name="BIGMAN_RIGHT_HAND" value="true" />
     <xacro:property name="BIGMAN_TORSO" value="true" />
     <xacro:property name="BIGMAN_LEFT_LEG" value="false" />
@@ -41,10 +41,10 @@
     <xacro:if value="${BIGMAN_LEFT_HAND}">
         <group name="left_hand">
-            <chain base_link="LWrMot3" tip_link="LSoftHandLink"/>
+            <chain base_link="LWrMot3" tip_link="LSoftHand"/>
         </group>
     </xacro:if>
     <xacro:if value="${BIGMAN_RIGHT_HAND}">
         <group name="right_hand">
-            <chain base_link="RWrMot3" tip_link="RSoftHandLink"/>
+            <chain base_link="RWrMot3" tip_link="RSoftHand"/>
         </group>
     </xacro:if>

File: IXBotInterface/configs/urdf/bigman_upper_body.urdf (robot description, URDF)
Before this commit: robot bigman, 55 links, 54 joints
Links:
- removed link LSoftHandLink
- removed link RSoftHandLink
- removed link TCP_L
- removed link TCP_R
- removed link l_hand_lower_left_link
- removed link l_hand_lower_right_link
- removed link l_hand_upper_left_link
- removed link l_hand_upper_right_link
- removed link r_hand_lower_left_link
- removed link r_hand_lower_right_link
- removed link r_hand_upper_left_link
- removed link r_hand_upper_right_link
- link LSoftHand: mass None -> 1.2; geometry collision box size=0.07 0.07 0.07; visual box size=0.07 0.07 0.07
- link RSoftHand: mass None -> 1.2; geometry collision box size=0.07 0.07 0.07; visual box size=0.07 0.07 0.07
Joints:
- removed joint TCP_Ljoint
- removed joint TCP_Rjoint
- removed joint l_handj2
- removed joint l_handj3
- removed joint l_handj4
- removed joint l_handj5
- removed joint l_handj6
- removed joint r_handj2
- removed joint r_handj3
- removed joint r_handj4
- removed joint r_handj5
- removed joint r_handj6
- joint l_handj: axis (none) -> -1 0 0; child LSoftHandLink -> LSoftHand; limit (none) -> lower=0 upper=5.0 effort=5 velocity=4.0; origin xyz=0 0 0 rpy=0 0 0 -> xyz=0 0 -0.04 rpy=0 0 0; type fixed -> revolute
- joint r_handj: axis (none) -> 1 0 0; child RSoftHandLink -> RSoftHand; limit (none) -> lower=0.0 upper=5.0 effort=5 velocity=4.0; origin xyz=0 0 0 rpy=0 0 0 -> xyz=0 0 -0.04 rpy=0 0 0; type fixed -> revolute
