Commit message: Bugfix concerning IMU loading

File: configs/urdf/centauro_upperbody.urdf (robot description, URDF)
Before this commit: robot centauro, 17 links, 16 joints
Links:
- added link test_imu_1, mass 0.0001
- added link test_imu_2, mass 0.0001
Joints:
- added joint test_imu_1_joint: type fixed, parent arm1_7, child test_imu_1, origin xyz=0.0 0.0 0.0, axis 0.1 -0.2 0.3
- added joint test_imu_2_joint: type fixed, parent arm2_7, child test_imu_2, origin xyz=0.0 0.0 0.0, axis 0.1 -0.2 0.3
